File: SensorHub/SensorHub/SensorHub.kicad_sch (KiCad schematic)
At the start: 90 parts, among them IC1 BMI088, J1 1-776087-1, J2 Conn_01x05_Pin, J3 USB_C_Receptacle_USB2.0_14P, SW1 SW_Push, U1 LMR33630ADDA, U2 TPS563200, U3 TPS7A2033PDBVR, U4 STM32L496RGT6, U5 TCAN330, U6 TCAN330, U7 USBLC6-2SC6, Y1 Crystal_GND24

Commit message: Arreglo conexion CAN2
Connections:
- net CAN2_RX: now also U6.4 (RXD)
- net CAN2_TX: now also U6.1 (TXD)
Changed lines of the file:
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@@
+	(wire
+		(pts
+			(xy 46.99 250.19) (xy 59.69 250.19)
+		)
+		(stroke
+			(width 0)
+			(type default)
+		)
+	)
 	(wire
 		(pts
@@
 		)
 		(stroke
+			(width 0)
+			(type default)
+		)
+	)
+	(wire
+		(pts
+			(xy 46.99 252.73) (xy 59.69 252.73)
+		)
+		(stroke
